File: ECUPrototypeIO/ECUPrototypeIO/conditioning_board.sch (KiCad schematic (older format))
At the start: 35 parts, among them J1 ECU Connector 1, J2 ECU Connector 2, J3 Relay Module Con2, J4 Vehicle Connector 1, J5 Relay Module Con1, Q1 MOSFET_A, SW1 MomentarySwitch, SW2 MomentarySwitch, U1 OPAmpA, U2 OPAmpB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

Commit message: latest files from jb laptop, unsure what changes exist
Parts:
- removed U1: LM358, symbol Amplifier_Operational:LM358
- removed U2: OPAmpB, symbol Amplifier_Operational:LM358
- removed U3: OPAmpC, symbol Amplifier_Operational:LM358
- added U? (x4): LM324, symbol Amplifier_Operational:LM324
- gave numbers to parts that had none: 8
Connections:
- net +12V: now also U?.4 (V+)
- net BrakeHBridge: now also U?.1
- net GND: now also U?.11 (V-)
- net RelayC_NO: now also U?.8
- net SteeringDriverConnector1_Yellow: now also U?.7
- net at C1.1, R4.1: now also U?.5 (+)
- net at R5.2, R6.1: now also U?.6 (-)
- net at C2.1, R9.1: now also U?.10 (+)
- net at R10.1, R11.2: now also U?.9 (-)
- net at C5.1, R16.1: now also U?.3 (+)
- net at R17.2, R18.1: now also U?.2 (-)
Changed lines of the file:
@@
-	1    0    0    -1
-$EndComp
-$Comp
-L Amplifier_Operational:LM358 U2
-U 1 1 5DE776D3
-P 9000 1850
-F 0 "U2" H 9000 2217 50  0000 C CNN
-F 1 "OPAmpB" H 9000 2126 50  0000 C CNN
-F 2 "" H 9000 1850 50  0001 C CNN
-F 3 "http://www.ti.com/lit/ds/symlink/lm2904-n.pdf" H 9000 1850 50  0001 C CNN
-	1    9000 1850
 	1    0    0    -1
 $EndComp
@@
 Connection ~ 8150 2450
 $Comp
-L Amplifier_Operational:LM358 U1
-U 3 1 5DE9087E
-P 9250 2450
-F 0 "U1" H 9208 2496 50  0000 L CNN
-F 1 "LM358" H 9208 2405 50  0000 L CNN
-F 2 "" H 9250 2450 50  0001 C CNN
-F 3 "http://www.ti.com/lit/ds/symlink/lm2904-n.pdf" H 9250 2450 50  0001 C CNN
-	3    9250 2450
-	0    1    1    0
-$EndComp
-$Comp
 L power:+12V #PWR0106
 U 1 1 5DEAC903
-P 9550 2350
-F 0 "#PWR0106" H 9550 2200 50  0001 C CNN
-F 1 "+12V" V 9565 2478 50  0000 L CNN
-F 2 "" H 9550 2350 50  0001 C CNN
-F 3 "" H 9550 2350 50  0001 C CNN
-	1    9550 2350
-	-1   0    0    1
+P 7000 2300
+F 0 "#PWR0106" H 7000 2150 50  0001 C CNN
+F 1 "+12V" V 7015 2428 50  0000 L CNN
+F 2 "" H 7000 2300 50  0001 C CNN
+F 3 "" H 7000 2300 50  0001 C CNN
+	1    7000 2300
+	1    0    0    -1
 $EndComp
 $Comp
 L power:GND #PWR0107
 U 1 1 5DEADCCD
-P 8950 2350
-F 0 "#PWR0107" H 8950 2100 50  0001 C CNN
-F 1 "GND" V 8955 2222 50  0000 R CNN
-F 2 "" H 8950 2350 50  0001 C CNN
-F 3 "" H 8950 2350 50  0001 C CNN
-	1    8950 2350
+P 7000 2900
+F 0 "#PWR0107" H 7000 2650 50  0001 C CNN
+F 1 "GND" V 7005 2772 50  0000 R CNN
+F 2 "" H 7000 2900 50  0001 C CNN
+F 3 "" H 7000 2900 50  0001 C CNN
+	1    7000 2900
 	1    0    0    -1
 $EndComp
@@
 	1    0    0    -1
 $EndComp
-$Comp
-L Amplifier_Operational:LM358 U1
-U 1 1 5DFCF209
-P 3450 2050
-F 0 "U1" H 3450 2417 50  0000 C CNN
-F 1 "OPAmpA" H 3450 2326 50  0000 C CNN
-F 2 "" H 3450 2050 50  0001 C CNN
-F 3 "http://www.ti.com/lit/ds/symlink/lm2904-n.pdf" H 3450 2050 50  0001 C CNN
-	1    3450 2050
-	1    0    0    -1
-$EndComp
 Wire Wire Line
 	2600 2650 2600 2700
@@
 RelayC_NO
 $Comp
-L power:GND #PWR?
+L power:GND #PWR03
 U 1 1 5E321D34
 P 3350 5350
-F 0 "#PWR?" H 3350 5100 50  0001 C CNN
+F 0 "#PWR03" H 3350 5100 50  0001 C CNN
 F 1 "GND" V 3355 5222 50  0000 R CNN
 F 2 "" H 3350 5350 50  0001 C CNN
@@
 $EndComp
 $Comp
-L power:+5V #PWR?
+L power:+5V #PWR02
 U 1 1 5E421138
 P 3300 4450
-F 0 "#PWR?" H 3300 4300 50  0001 C CNN
+F 0 "#PWR02" H 3300 4300 50  0001 C CNN
 F 1 "+5V" H 3315 4623 50  0000 C CNN
 F 2 "" H 3300 4450 50  0001 C CNN
@@
 Text GLabel 13450 5750 0    50   Input ~ 0
 MotorSpeed_Red
-$Comp
-L Amplifier_Operational:LM358 U3
-U 1 1 5E8DD5BA
-P 3450 3400
-F 0 "U3" H 3450 3767 50  0000 C CNN
-F 1 "OPAmpC" H 3450 3676 50  0000 C CNN
-F 2 "" H 3450 3400 50  0001 C CNN
-F 3 "http://www.ti.com/lit/ds/symlink/lm2904-n.pdf" H 3450 3400 50  0001 C CNN
-	1    3450 3400
-	1    0    0    -1
-$EndComp
 Wire Wire Line
 	2600 3300 3150 3300
@@
 	8350 4800 7950 4800
 $Comp
-L power:GNDA #PWR?
+L power:GNDA #PWR07
 U 1 1 5E94E013
 P 8350 5100
-F 0 "#PWR?" H 8350 4850 50  0001 C CNN
+F 0 "#PWR07" H 8350 4850 50  0001 C CNN
 F 1 "GNDA" H 8355 4927 50  0000 C CNN
 F 2 "" H 8350 5100 50  0001 C CNN
@@
 	8350 4800 8650 4800
 $Comp
-L Device:R R?
+L Device:R R12
 U 1 1 5E94E008
 P 8800 4800
-F 0 "R?" V 8593 4800 50  0000 C CNN
+F 0 "R12" V 8593 4800 50  0000 C CNN
 F 1 "10K" V 8684 4800 50  0000 C CNN
 F 2 "" V 8730 4800 50  0001 C CNN
@@
 $EndComp
 $Comp
-L Device:R R?
+L Device:R R7
 U 1 1 5E94DFFE
 P 8350 4950
-F 0 "R?" H 8420 4996 50  0000 L CNN
+F 0 "R7" H 8420 4996 50  0000 L CNN
 F 1 "20K" H 8420 4905 50  0000 L CNN
 F 2 "" V 8280 4950 50  0001 C CNN
@@
 	8200 3850 7800 3850
 $Comp
-L power:GNDA #PWR?
+L power:GNDA #PWR05
 U 1 1 5E9BDB3F
 P 8200 4150
-F 0 "#PWR?" H 8200 3900 50  0001 C CNN
+F 0 "#PWR05" H 8200 3900 50  0001 C CNN
 F 1 "GNDA" H 8205 3977 50  0000 C CNN
 F 2 "" H 8200 4150 50  0001 C CNN
@@
 	8200 3850 8500 3850
 $Comp
-L Device:R R?
+L Device:R R8
 U 1 1 5E9BDB4A
 P 8650 3850
-F 0 "R?" V 8443 3850 50  0000 C CNN
+F 0 "R8" V 8443 3850 50  0000 C CNN
 F 1 "10K" V 8534 3850 50  0000 C CNN
 F 2 "" V 8580 3850 50  0001 C CNN
@@
 $EndComp
 $Comp
-L Device:R R?
+L Device:R R3
 U 1 1 5E9BDB54
 P 8200 4000
-F 0 "R?" H 8270 4046 50  0000 L CNN
+F 0 "R3" H 8270 4046 50  0000 L CNN
 F 1 "20K" H 8270 3955 50  0000 L CNN
 F 2 "" V 8130 4000 50  0001 C CNN
@@
 $EndComp
 $Comp
-L power:GND #PWR?
+L power:GND #PWR01
 U 1 1 5EA112FB
 P 1850 7250
-F 0 "#PWR?" H 1850 7000 50  0001 C CNN
+F 0 "#PWR01" H 1850 7000 50  0001 C CNN
 F 1 "GND" V 1855 7122 50  0000 R CNN
 F 2 "" H 1850 7250 50  0001 C CNN
@@
 VehicleConnector2
 $Comp
-L Device:R R?
+L Device:R R1
 U 1 1 5EE5DE17
 P 7400 5700
-F 0 "R?" V 7193 5700 50  0000 C CNN
+F 0 "R1" V 7193 5700 50  0000 C CNN
 F 1 "R" V 7284 5700 50  0000 C CNN
 F 2 "" V 7330 5700 50  0001 C CNN
@@
 	7550 5700 7650 5700
 $Comp
-L Device:R R?
+L Device:R R2
 U 1 1 5EE6BE7F
 P 7650 6050
-F 0 "R?" H 7580 6004 50  0000 R CNN
+F 0 "R2" H 7580 6004 50  0000 R CNN
 F 1 "R" H 7580 6095 50  0000 R CNN
 F 2 "" V 7580 6050 50  0001 C CNN
@@
 	7650 6200 7650 6300
 $Comp
-L power:GND #PWR?
+L power:GND #PWR04
 U 1 1 5EE72182
 P 7650 6300
-F 0 "#PWR?" H 7650 6050 50  0001 C CNN
+F 0 "#PWR04" H 7650 6050 50  0001 C CNN
 F 1 "GND" H 7655 6127 50  0000 C CNN
 F 2 "" H 7650 6300 50  0001 C CNN
@@
 Connection ~ 7650 5700
 $Comp
-L Device:C C?
+L Device:C C3
 U 1 1 5EE8749A
 P 8200 6100
-F 0 "C?" H 8315 6146 50  0000 L CNN
+F 0 "C3" H 8315 6146 50  0000 L CNN
 F 1 "C" H 8315 6055 50  0000 L CNN
 F 2 "" H 8238 5950 50  0001 C CNN
@@
 	8200 5700 8200 5950
 $Comp
-L power:GND #PWR?
+L power:GND #PWR06
 U 1 1 5EE903F0
 P 8200 6300
-F 0 "#PWR?" H 8200 6050 50  0001 C CNN
+F 0 "#PWR06" H 8200 6050 50  0001 C CNN
 F 1 "GND" H 8205 6127 50  0000 C CNN
 F 2 "" H 8200 6300 50  0001 C CNN
@@
 	9950 5700 10150 5700
 $Comp
-L power:GND #PWR?
+L power:GND #PWR08
 U 1 1 5EE9E693
 P 8550 6550
-F 0 "#PWR?" H 8550 6300 50  0001 C CNN
+F 0 "#PWR08" H 8550 6300 50  0001 C CNN
 F 1 "GND" H 8555 6377 50  0000 C CNN
 F 2 "" H 8550 6550 50  0001 C CNN
@@
 	8350 5700 9100 5700
 $Comp
-L 74xx:74LS14 U?
+L 74xx:74LS14 U4
 U 1 1 5EEA2972
 P 9400 5700
-F 0 "U?" H 9400 6017 50  0000 C CNN
+F 0 "U4" H 9400 6017 50  0000 C CNN
 F 1 "74LS14" H 9400 5926 50  0000 C CNN
 F 2 "" H 9400 5700 50  0001 C CNN
@@
 $EndComp
 $Comp
-L 74xx:74LS14 U?
+L 74xx:74LS14 U4
 U 7 1 5EEC9705
 P 9050 6150
-F 0 "U?" V 8683 6150 50  0000 C CNN
+F 0 "U4" V 8683 6150 50  0000 C CNN
 F 1 "74LS14" V 8774 6150 50  0000 C CNN
 F 2 "" H 9050 6150 50  0001 C CNN
@@
 	8550 6150 8550 6550
 $Comp
-L power:+5V #PWR?
+L power:+5V #PWR09
 U 1 1 5EEED749
 P 9550 6500
-F 0 "#PWR?" H 9550 6350 50  0001 C CNN
+F 0 "#PWR09" H 9550 6350 50  0001 C CNN
 F 1 "+5V" H 9565 6673 50  0000 C CNN
 F 2 "" H 9550 6500 50  0001 C CNN
@@
 Wire Notes Line
 	6200 1000 6200 7100
+$Comp
+L Amplifier_Operational:LM324 U?
+U 1 1 5E651428
+P 3450 2050
+F 0 "U?" H 3450 2417 50  0000 C CNN
+F 1 "LM324" H 3450 2326 50  0000 C CNN
+F 2 "" H 3400 2150 50  0001 C CNN
+F 3 "http://www.ti.com/lit/ds/symlink/lm2902-n.pdf" H 3500 2250 50  0001 C CNN
+	1    3450 2050
+	1    0    0    -1
+$EndComp
+$Comp
+L Amplifier_Operational:LM324 U?
+U 2 1 5E6564AD
+P 9000 1850
+F 0 "U?" H 9000 2217 50  0000 C CNN
+F 1 "LM324" H 9000 2126 50  0000 C CNN
+F 2 "" H 8950 1950 50  0001 C CNN
+F 3 "http://www.ti.com/lit/ds/symlink/lm2902-n.pdf" H 9050 2050 50  0001 C CNN
+	2    9000 1850
+	1    0    0    -1
+$EndComp
+$Comp
+L Amplifier_Operational:LM324 U?
+U 3 1 5E65A543
+P 3450 3400
+F 0 "U?" H 3450 3767 50  0000 C CNN
+F 1 "LM324" H 3450 3676 50  0000 C CNN
+F 2 "" H 3400 3500 50  0001 C CNN
+F 3 "http://www.ti.com/lit/ds/symlink/lm2902-n.pdf" H 3500 3600 50  0001 C CNN
+	3    3450 3400
+	1    0    0    -1
+$EndComp
+$Comp
+L Amplifier_Operational:LM324 U?
+U 5 1 5E65CD8B
+P 7100 2600
+F 0 "U?" H 7058 2646 50  0000 L CNN
+F 1 "LM324" H 7058 2555 50  0000 L CNN
+F 2 "" H 7050 2700 50  0001 C CNN
+F 3 "http://www.ti.com/lit/ds/symlink/lm2902-n.pdf" H 7150 2800 50  0001 C CNN
+	5    7100 2600
+	1    0    0    -1
+$EndComp
 $EndSCHEMATC
