File: ECUPrototypeIO/ECUPrototypeIO/ECUProtoypeIO/ECUPrototypeIO - Copy.sch (KiCad schematic (older format))
At the start: 35 parts, among them SW2 MomentarySwitch, U1 LM358

Commit message: Cleaned Up Diagram, Added I/O Spreadsheet for Diagnostics and Validation
Parts:
- removed R? (x2): R, symbol pspice:R
Connections:
- wire segments 153 -> 150
Other:
- moved on the sheet: R14, R15
Changed lines of the file:
@@
 Wire Wire Line
 	7750 4100 8100 4100
-Text GLabel 8350 5000 0    50   Input ~ 0
+Text GLabel 7750 2700 0    50   Input ~ 0
 ESTOP
 $Comp
 L Device:R R14
 U 1 1 5DE1B463
-P 8750 5150
-F 0 "R14" H 8820 5196 50  0000 L CNN
-F 1 "39K" H 8820 5105 50  0000 L CNN
-F 2 "" V 8680 5150 50  0001 C CNN
-F 3 "~" H 8750 5150 50  0001 C CNN
-	1    8750 5150
+P 8150 2850
+F 0 "R14" H 8220 2896 50  0000 L CNN
+F 1 "39K" H 8220 2805 50  0000 L CNN
+F 2 "" V 8080 2850 50  0001 C CNN
+F 3 "~" H 8150 2850 50  0001 C CNN
+	1    8150 2850
 	1    0    0    -1
 $EndComp
@@
 L Device:R R15
 U 1 1 5DE1C159
-P 9200 5000
-F 0 "R15" V 8993 5000 50  0000 C CNN
-F 1 "10K" V 9084 5000 50  0000 C CNN
-F 2 "" V 9130 5000 50  0001 C CNN
-F 3 "~" H 9200 5000 50  0001 C CNN
-	1    9200 5000
-	0    1    1    0
-$EndComp
-Wire Wire Line
-	8750 5000 9050 5000
+P 8600 2700
+F 0 "R15" V 8393 2700 50  0000 C CNN
+F 1 "10K" V 8484 2700 50  0000 C CNN
+F 2 "" V 8530 2700 50  0001 C CNN
+F 3 "~" H 8600 2700 50  0001 C CNN
+	1    8600 2700
+	0    1    1    0
+$EndComp
+Wire Wire Line
+	8150 2700 8450 2700
 $Comp
 L power:GNDA #PWR0117
 U 1 1 5DE24ED1
-P 8750 5300
-F 0 "#PWR0117" H 8750 5050 50  0001 C CNN
-F 1 "GNDA" H 8755 5127 50  0000 C CNN
-F 2 "" H 8750 5300 50  0001 C CNN
-F 3 "" H 8750 5300 50  0001 C CNN
-	1    8750 5300
-	1    0    0    -1
-$EndComp
-Wire Wire Line
-	8750 5000 8350 5000
-Connection ~ 8750 5000
-Text GLabel 9550 5000 2    50   Input ~ 0
+P 8150 3000
+F 0 "#PWR0117" H 8150 2750 50  0001 C CNN
+F 1 "GNDA" H 8155 2827 50  0000 C CNN
+F 2 "" H 8150 3000 50  0001 C CNN
+F 3 "" H 8150 3000 50  0001 C CNN
+	1    8150 3000
+	1    0    0    -1
+$EndComp
+Wire Wire Line
+	8150 2700 7750 2700
+Connection ~ 8150 2700
+Text GLabel 8950 2700 2    50   Input ~ 0
 ESTOP_In
 Wire Wire Line
-	9550 5000 9350 5000
+	8950 2700 8750 2700
 Wire Wire Line
 	4500 2100 4250 2100
@@
 Wire Wire Line
 	3550 3000 3900 3000
-Wire Wire Line
-	7050 6250 7000 6250
 Text GLabel 4500 1550 2    50   Input ~ 0
 RelayModuleGnd
@@
 Wire Wire Line
 	2050 1650 2050 1700
-Connection ~ 2050 1700
-Wire Wire Line
-	2050 1700 2050 1850
 Wire Wire Line
 	7500 3800 8100 3800
@@
 	10550 1400 10250 1400
 Connection ~ 10250 1400
-$Comp
-L pspice:R R?
-U 1 1 5EAC0A55
-P 10450 2400
-F 0 "R?" V 10245 2400 50  0000 C CNN
-F 1 "R" V 10336 2400 50  0000 C CNN
-F 2 "" H 10450 2400 50  0001 C CNN
-F 3 "~" H 10450 2400 50  0001 C CNN
-	1    10450 2400
-	0    1    1    0
-$EndComp
 Wire Wire Line
 	11250 2050 11250 2400
-Wire Wire Line
-	11250 2400 10700 2400
-Wire Wire Line
-	10200 2400 10200 2500
-$Comp
-L pspice:R R?
-U 1 1 5EAE5FA7
-P 10200 2750
-F 0 "R?" H 10132 2704 50  0000 R CNN
-F 1 "R" H 10132 2795 50  0000 R CNN
-F 2 "" H 10200 2750 50  0001 C CNN
-F 3 "~" H 10200 2750 50  0001 C CNN
-	1    10200 2750
-	-1   0    0    1
-$EndComp
-$Comp
-L power:GND #PWR?
-U 1 1 5EAE73F7
-P 10200 3000
-F 0 "#PWR?" H 10200 2750 50  0001 C CNN
-F 1 "GND" V 10205 2872 50  0000 R CNN
-F 2 "" H 10200 3000 50  0001 C CNN
-F 3 "" H 10200 3000 50  0001 C CNN
-	1    10200 3000
-	1    0    0    -1
-$EndComp
 Text GLabel 11250 2800 0    50   Input ~ 0
 SafetyLights1
@@
 	11250 2400 11250 2800
 Connection ~ 11250 2400
-Wire Wire Line
-	10200 2400 9900 2400
-Connection ~ 10200 2400
 Text GLabel 9900 2400 0    50   Input ~ 0
 EstopIN
@@
 	-1   0    0    1
 $EndComp
+Text GLabel 11650 2350 2    50   Input ~ 0
+RelayModuleGnd
+Wire Wire Line
+	11650 2050 11650 2350
+Wire Wire Line
+	9900 2400 11250 2400
 $EndSCHEMATC

Commit message: Updates to I.O Spreadsheet
Connections:
- net EstopIN is gone; now on net ESTOP_In: B.7, B.8
Changed lines of the file:
@@
 Connection ~ 11250 2400
 Text GLabel 9900 2400 0    50   Input ~ 0
-EstopIN
+ESTOP_In
 Wire Wire Line
 	7400 1550 6600 1550
