File: ECUPrototypeIO/ECUPrototypeIO/ConditioningBoard/CB3/CB3/CB3.sch (KiCad schematic (older format))
At the start: 28 parts, among them J1 ECU Connector 1, J2 ECU Connector 2, J3 Relay Module Con2, J4 Vehicle Connector 1, J5 Relay Module Con1, Q1 MOSFET_A, SW1 MomentarySwitch, SW2 MomentarySwitch, T1 Screw_Terminal_01x04, U1 LM324

Commit message: grouped relevant components on PCB Schematic
Changed lines of the file:
@@
 	11350 1000 6200 1000
 Text Label 8500 1200 0    50   ~ 0
-VehicleConnector2
+ECUConnector2
 $Comp
 L Device:R R1

Commit message: latest files from jb laptop, unsure what changes exist
Parts:
- removed Q1: MOSFET_A, Package_TO_SOT_THT:TO-220-3_Vertical, symbol Transistor_FET:IRLZ44N
- removed unit 3 of U1
- added D1: 3.3V, Diode_THT:D_T-1_P5.08mm_Horizontal, symbol Diode:1N47xxA
- added D2: 1N4001, Diode_THT:D_DO-41_SOD81_P10.16mm_Horizontal, symbol Diode:1N4001
- added D3: 5.6V, Diode_THT:D_T-1_P5.08mm_Horizontal, symbol Diode:1N47xxA
- added D4, D5: LD271, LED_THT:LED_D5.0mm_IRGrey, symbol LED:LD271
- added F1: 1A Fuse, Fuse:Fuse_0805_2012Metric, symbol Device:Fuse_Small
- added Q1: 2N7002H, Package_TO_SOT_SMD:SOT-23, symbol Transistor_FET:2N7002H
- added R16: 330, Resistor_THT:R_Axial_DIN0207_L6.3mm_D2.5mm_P10.16mm_Horizontal, symbol Device:R
- added R17: 1K, Resistor_THT:R_Axial_DIN0207_L6.3mm_D2.5mm_P10.16mm_Horizontal, symbol Device:R
- added unit 1 of U1
- J1, J2, J3: symbol Connector:DB9_Female -> Connector:DB9_Female_MountingHoles
- J4, J5: symbol Connector:DB9_Male -> Connector:DB9_Male_MountingHoles
- R12, R8: value 10K -> 220K
- R3, R7: value 20K -> 330K
Connections:
- net AccelerationEnable: now also Q1.1 (G)
- net GND: now also J1.0 (PAD), J2.0 (PAD), J3.0 (PAD), J4.0 (PAD), J5.0 (PAD), D1.2 (A), D3.2 (A), Q1.2 (S), R16.2, R17.2
- net MotorSpeed_Red: now also D2.2 (A); no longer R1.1, R2.2
- net RelayC_NO: now also U1.1
- net RelayD_NO: now also Q1.3 (D)
- net VehicleSpeed: now also D1.1 (K)
- net at C2.1, R9.1: now also U1.3 (+)
- net at R10.1, R11.2: now also U1.2 (-)
- net +12V renamed 12V
- net 12V: now also D5.2 (A)
- net +5V renamed 5V_Fused
- net 5V_Fused: now also D3.1 (K), D4.2 (A), F1.1; no longer T1.4 (Pin_4)
- new net: D4.1 (K), R16.1
- new net: D5.1 (K), R17.1
- new net: D2.1 (K), R1.1, R2.2
- new net 5V: F1.2, T1.4 (Pin_4)

Commit message: Look at README File
Parts:
- C1, C2, C3: footprint Capacitor_SMD:C_0805_2012Metric -> Capacitor_THT:C_Disc_D7.5mm_W5.0mm_P7.50mm
- F1: footprint Fuse:Fuse_0805_2012Metric -> Fuse:Fuse_Littelfuse-LVR100
- Q1: footprint Package_TO_SOT_SMD:SOT-23 -> Package_TO_SOT_THT:SIPAK-1EP_Horizontal_TabDown
Other:
- note added: "OPEN ERRORS:\n\n- Op-Amp gain error?\n (Need function generator to test)\n- Verify mosfet circuit"
- note added: "OPEN ERRORS:\n\n- Op-Amp gain error?\n- Voltage divider only drops 12V to 9.5V \n (Vd_c is Vin, Estop is Vout)"
Changed lines of the file:
@@
 F 0 "C1" H 8265 2146 50  0000 L CNN
 F 1 "100nF" H 8265 2055 50  0000 L CNN
-F 2 "Capacitor_SMD:C_0805_2012Metric" H 8188 1950 50  0001 C CNN
+F 2 "Capacitor_THT:C_Disc_D7.5mm_W5.0mm_P7.50mm" H 8188 1950 50  0001 C CNN
 F 3 "~" H 8150 2100 50  0001 C CNN
 	1    8150 2100
@@
 F 0 "C2" H 2715 3696 50  0000 L CNN
 F 1 "100nF" H 2715 3605 50  0000 L CNN
-F 2 "Capacitor_SMD:C_0805_2012Metric" H 2638 3500 50  0001 C CNN
+F 2 "Capacitor_THT:C_Disc_D7.5mm_W5.0mm_P7.50mm" H 2638 3500 50  0001 C CNN
 F 3 "~" H 2600 3650 50  0001 C CNN
 	1    2600 3650
@@
 F 0 "C3" H 8765 6146 50  0000 L CNN
 F 1 "100nF" H 8765 6055 50  0000 L CNN
-F 2 "Capacitor_SMD:C_0805_2012Metric" H 8688 5950 50  0001 C CNN
+F 2 "Capacitor_THT:C_Disc_D7.5mm_W5.0mm_P7.50mm" H 8688 5950 50  0001 C CNN
 F 3 "~" H 8650 6100 50  0001 C CNN
 	1    8650 6100
@@
 F 0 "Q1" H 3455 5046 50  0000 L CNN
 F 1 "2N7002H" H 3455 4955 50  0000 L CNN
-F 2 "Package_TO_SOT_SMD:SOT-23" H 3450 4925 50  0001 L CIN
+F 2 "Package_TO_SOT_THT:SIPAK-1EP_Horizontal_TabDown" H 3450 4925 50  0001 L CIN
 F 3 "http://www.diodes.com/assets/Datasheets/2N7002H.pdf" H 3250 5000 50  0001 L CNN
 	1    3250 5000
@@
 F 0 "F1" H 1900 1735 50  0000 C CNN
 F 1 "1A Fuse" H 1900 1644 50  0000 C CNN
-F 2 "Fuse:Fuse_0805_2012Metric" H 1900 1550 50  0001 C CNN
+F 2 "Fuse:Fuse_Littelfuse-LVR100" H 1900 1550 50  0001 C CNN
 F 3 "~" H 1900 1550 50  0001 C CNN
 	1    1900 1550
@@
 Text GLabel 7000 2300 1    50   Input ~ 0
 12V
+Text Notes 9000 2750 0    50   ~ 10
+OPEN ERRORS:\n\n- Op-Amp gain error?\n- Voltage divider only drops 12V to 9.5V \n    (Vd_c is Vin, Estop is Vout)
+Text Notes 3700 4200 0    50   ~ 10
+OPEN ERRORS:\n\n- Op-Amp gain error?\n   (Need function generator to test)\n- Verify mosfet circuit
 $EndSCHEMATC

Commit message: Look at README
Parts:
- added R18: 10k, Resistor_THT:R_Axial_DIN0207_L6.3mm_D2.5mm_P10.16mm_Horizontal, symbol Device:R
Connections:
- net AccelerationEnable: now also R18.2
- net ESTOP: now also R14.2; no longer R14.1, R15.2
- net GND: now also R15.1, R18.1; no longer R14.2
- net VoltageDivider_C: now also R14.1, R15.2; no longer R15.1
Other:
- note added: "Modified:\n\n- Added pull down resistor to mosfet circuit"
- note added: "Modified\n\n- Flipped resistors Vdc to ESTOP voltage divider"
- note removed: "OPEN ERRORS:\n\n- Op-Amp gain error?\n (Need function generator to test)\n- Verify mosfet circuit"
- note removed: "OPEN ERRORS:\n\n- Op-Amp gain error?\n- Voltage divider only drops 12V to 9.5V \n (Vd_c is Vin, Estop is Vout)"
Changed lines of the file:
@@
 	9400 1850 9950 1850
 Connection ~ 9400 1850
-Text GLabel 7800 3100 0    50   Input ~ 0
+Text GLabel 7700 3000 0    50   Input ~ 0
 ESTOP
-$Comp
-L Device:R R14
-U 1 1 5DE1B463
-P 8200 3250
-F 0 "R14" H 8270 3296 50  0000 L CNN
-F 1 "39K" H 8270 3205 50  0000 L CNN
-F 2 "Resistor_THT:R_Axial_DIN0207_L6.3mm_D2.5mm_P10.16mm_Horizontal" V 8130 3250 50  0001 C CNN
-F 3 "~" H 8200 3250 50  0001 C CNN
-	1    8200 3250
-	1    0    0    -1
-$EndComp
-$Comp
-L Device:R R15
-U 1 1 5DE1C159
-P 8650 3100
-F 0 "R15" V 8443 3100 50  0000 C CNN
-F 1 "10K" V 8534 3100 50  0000 C CNN
-F 2 "Resistor_THT:R_Axial_DIN0207_L6.3mm_D2.5mm_P10.16mm_Horizontal" V 8580 3100 50  0001 C CNN
-F 3 "~" H 8650 3100 50  0001 C CNN
-	1    8650 3100
-	0    1    1    0
-$EndComp
-Wire Wire Line
-	8200 3100 8500 3100
-$Comp
-L power:GNDA #PWR0117
-U 1 1 5DE24ED1
-P 8200 3400
-F 0 "#PWR0117" H 8200 3150 50  0001 C CNN
-F 1 "GNDA" H 8205 3227 50  0000 C CNN
-F 2 "" H 8200 3400 50  0001 C CNN
-F 3 "" H 8200 3400 50  0001 C CNN
-	1    8200 3400
-	1    0    0    -1
-$EndComp
-Wire Wire Line
-	8200 3100 7800 3100
-Connection ~ 8200 3100
-Text GLabel 9000 3100 2    50   Input ~ 0
+Text GLabel 8900 3000 2    50   Input ~ 0
 VoltageDivider_C
-Wire Wire Line
-	9000 3100 8800 3100
 Text GLabel 5600 8550 0    50   Input ~ 0
 GND
@@
 L power:GND #PWR03
 U 1 1 5E321D34
-P 3350 5350
-F 0 "#PWR03" H 3350 5100 50  0001 C CNN
-F 1 "GND" V 3355 5222 50  0000 R CNN
-F 2 "" H 3350 5350 50  0001 C CNN
-F 3 "" H 3350 5350 50  0001 C CNN
-	1    3350 5350
-	1    0    0    -1
-$EndComp
-Wire Wire Line
-	2550 5000 3050 5000
+P 3350 5400
+F 0 "#PWR03" H 3350 5150 50  0001 C CNN
+F 1 "GND" V 3355 5272 50  0000 R CNN
+F 2 "" H 3350 5400 50  0001 C CNN
+F 3 "" H 3350 5400 50  0001 C CNN
+	1    3350 5400
+	1    0    0    -1
+$EndComp
+Wire Wire Line
+	2550 5000 2900 5000
 Wire Wire Line
 	3300 4750 3300 4800
@@
 12V
 Text Notes 9000 2750 0    50   ~ 10
-OPEN ERRORS:\n\n- Op-Amp gain error?\n- Voltage divider only drops 12V to 9.5V \n    (Vd_c is Vin, Estop is Vout)
+Modified\n\n- Flipped resistors Vdc to ESTOP voltage divider
 Text Notes 3700 4200 0    50   ~ 10
-OPEN ERRORS:\n\n- Op-Amp gain error?\n   (Need function generator to test)\n- Verify mosfet circuit
+Modified:\n\n- Added pull down resistor to mosfet circuit
+$Comp
+L Device:R R18
+U 1 1 5F69E7D0
+P 2900 5200
+F 0 "R18" V 2693 5200 50  0000 C CNN
+F 1 "10k" V 2784 5200 50  0000 C CNN
+F 2 "Resistor_THT:R_Axial_DIN0207_L6.3mm_D2.5mm_P10.16mm_Horizontal" V 2830 5200 50  0001 C CNN
+F 3 "~" H 2900 5200 50  0001 C CNN
+	1    2900 5200
+	-1   0    0    1
+$EndComp
+Wire Wire Line
+	2900 5050 2900 5000
+Connection ~ 2900 5000
+Wire Wire Line
+	2900 5000 3050 5000
+Wire Wire Line
+	2900 5350 3350 5350
+Connection ~ 3350 5350
+Wire Wire Line
+	3350 5350 3350 5400
+$Comp
+L Device:R R15
+U 1 1 5F6C5EC2
+P 8450 3200
+F 0 "R15" V 8243 3200 50  0000 C CNN
+F 1 "10K" V 8334 3200 50  0000 C CNN
+F 2 "Resistor_THT:R_Axial_DIN0207_L6.3mm_D2.5mm_P10.16mm_Horizontal" V 8380 3200 50  0001 C CNN
+F 3 "~" H 8450 3200 50  0001 C CNN
+	1    8450 3200
+	-1   0    0    1
+$EndComp
+$Comp
+L Device:R R14
+U 1 1 5F6C70BA
+P 8150 3000
+F 0 "R14" H 8220 3046 50  0000 L CNN
+F 1 "39K" H 8220 2955 50  0000 L CNN
+F 2 "Resistor_THT:R_Axial_DIN0207_L6.3mm_D2.5mm_P10.16mm_Horizontal" V 8080 3000 50  0001 C CNN
+F 3 "~" H 8150 3000 50  0001 C CNN
+	1    8150 3000
+	0    1    1    0
+$EndComp
+Wire Wire Line
+	8900 3000 8450 3000
+Wire Wire Line
+	8450 3050 8450 3000
+Connection ~ 8450 3000
+Wire Wire Line
+	8450 3000 8300 3000
+Wire Wire Line
+	8000 3000 7700 3000
+$Comp
+L power:GNDA #PWR0103
+U 1 1 5F70057C
+P 8450 3400
+F 0 "#PWR0103" H 8450 3150 50  0001 C CNN
+F 1 "GNDA" H 8455 3227 50  0000 C CNN
+F 2 "" H 8450 3400 50  0001 C CNN
+F 3 "" H 8450 3400 50  0001 C CNN
+	1    8450 3400
+	1    0    0    -1
+$EndComp
+Wire Wire Line
+	8450 3350 8450 3400
 $EndSCHEMATC
